File: GlowHubPCB/GlowHubPCB.kicad_pcb (KiCad board)
At the start: 2 copper layers, 43.4 x 82.8 mm, 47 parts, among them J1 Conn_01x08, Q1 AP40P05, Q10 AP40P05, Q11 AP40P05, Q2 MMBT2222A, Q3 MMBT2222A, Q4 AP40P05, Q5 AP40P05, Q6 AP40P05, Q7 AP40P05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

Commit message: updated pcb design (in progress)
Parts:
- SW1, SW2: value SW-SMD_4P-L3.7-W3.0-P1.50-LS4.7 -> TS-1185EC-C-D-B
- U5: value Val** -> CP2102-GMR
Connections:
- Q3 pad 2: RESET -> RTS
- Q3 pad 3: RTS -> RESET
Routing:
- net RESET: track 76.4 -> 77.3 mm
- net RTS: track 28.6 -> 29.3 mm
Changed lines of the file:
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@@
   (net 95 "EXTERNAL 5V")
   (net 96 "Net-(C17-Pad2)")
-  (net 97 "Net-(USB1-PadA4B9)")
+  (net 97 "Net-(F1-Pad1)")
   (footprint "Package_TO_SOT_SMD:SOT-23" (layer "F.Cu")
     (at 56.471 53.7346)
@@
       (effects (font (size 1 1) (thickness 0.15)))
     )
-    (fp_text value "SW-SMD_4P-L3.7-W3.0-P1.50-LS4.7" (at 0 4.75) (layer "F.Fab")
+    (fp_text value "TS-1185EC-C-D-B" (at 0 4.75) (layer "F.Fab")
       (effects (font (size 1 1) (thickness 0.15)))
     )
@@
     (property "Sheetfile" "GlowHubPCB.kicad_sch")
     (property "Sheetname" "")
-    (attr through_hole exclude_from_pos_files exclude_from_bom)
+    (attr through_hole exclude_from_pos_files)
     (fp_text reference "J1" (at 0 -2.77 90) (layer "F.SilkS") hide
       (effects (font (size 1 1) (thickness 0.15)))
@@
       (net 29 "Net-(Q3-Pad1)") (pintype "passive"))
     (pad "2" smd roundrect (at -0.9375 0.95 270) (size 1.475 0.6) (layers "F.Cu" "F.Paste" "F.Mask") (roundrect_rratio 0.25)
-      (net 19 "RESET") (pintype "passive"))
-    (pad "3" smd roundrect (at 0.9375 0 270) (size 1.475 0.6) (layers "F.Cu" "F.Paste" "F.Mask") (roundrect_rratio 0.25)
       (net 32 "RTS") (pintype "passive"))
+    (pad "3" smd roundrect (at 0.9375 0 270) (size 1.475 0.6) (layers "F.Cu" "F.Paste" "F.Mask") (roundrect_rratio 0.25)
+      (net 19 "RESET") (pintype "passive"))
     (model "${KICAD6_3DMODEL_DIR}/Package_TO_SOT_SMD.3dshapes/SOT-23.step"
       (offset (xyz 0 0 0))
@@
       (net 1 "GND") (pinfunction "GND") (pintype "unspecified"))
     (pad "A4B9" smd rect locked (at -2.4 -2.46 270) (size 0.6 1.3) (layers "F.Cu" "F.Paste" "F.Mask")
-      (net 97 "Net-(USB1-PadA4B9)") (pinfunction "VBUS") (pintype "unspecified"))
+      (net 97 "Net-(F1-Pad1)") (pinfunction "VBUS") (pintype "unspecified"))
     (pad "A5" smd rect locked (at -1.25 -2.46 270) (size 0.3 1.3) (layers "F.Cu" "F.Paste" "F.Mask")
       (net 37 "USB-C CC1") (pinfunction "CC1") (pintype "unspecified"))
@@
       (net 1 "GND") (pinfunction "GND") (pintype "unspecified"))
     (pad "B4A9" smd rect locked (at 2.4 -2.46 270) (size 0.6 1.3) (layers "F.Cu" "F.Paste" "F.Mask")
-      (net 97 "Net-(USB1-PadA4B9)") (pinfunction "VBUS") (pintype "unspecified"))
+      (net 97 "Net-(F1-Pad1)") (pinfunction "VBUS") (pintype "unspecified"))
     (pad "B5" smd rect locked (at 1.75 -2.46 270) (size 0.3 1.3) (layers "F.Cu" "F.Paste" "F.Mask")
       (net 86 "USB-C CC2") (pinfunction "CC2") (pintype "unspecified"))
@@
       (effects (font (size 1 1) (thickness 0.15)))
     )
-    (fp_text value "SW-SMD_4P-L3.7-W3.0-P1.50-LS4.7" (at 0 4.75) (layer "F.Fab")
+    (fp_text value "TS-1185EC-C-D-B" (at 0 4.75) (layer "F.Fab")
       (effects (font (size 1 1) (thickness 0.15)))
     )
@@
       (effects (font (size 1 1) (thickness 0.15)) (justify left))
     )
-    (fp_text value "Val**" (at 0 0) (layer "F.SilkS") hide
+    (fp_text value "CP2102-GMR" (at 0 0) (layer "F.SilkS") hide
       (effects (font (size 1.27 1.27) (thickness 0.15)))
     )
@@
     (fp_line (start -2.25 -1.6) (end 2.25 -1.6) (layer "F.Fab") (width 0.1))
     (pad "1" smd roundrect (at -2.225 0) (size 1.3 3.4) (layers "F.Cu" "F.Paste" "F.Mask") (roundrect_rratio 0.1923076923)
-      (net 97 "Net-(USB1-PadA4B9)") (pintype "passive"))
+      (net 97 "Net-(F1-Pad1)") (pintype "passive"))
     (pad "2" smd roundrect (at 2.225 0) (size 1.3 3.4) (layers "F.Cu" "F.Paste" "F.Mask") (roundrect_rratio 0.1923076923)
       (net 31 "+5V") (pintype "passive"))
@@
   (segment (start 68.461 61.1146) (end 68.14805 60.80165) (width 0.16) (layer "F.Cu") (net 19))
   (segment (start 69.0385 123.4146) (end 69.0385 123.3021) (width 0.16) (layer "F.Cu") (net 19))
+  (segment (start 72.2966 93.865) (end 72.2966 94.7995) (width 0.16) (layer "F.Cu") (net 19))
+  (segment (start 72.2966 94.7995) (end 72.0261 95.07) (width 0.16) (layer "F.Cu") (net 19))
   (segment (start 72.456 122.9196) (end 71.381 121.8446) (width 0.16) (layer "F.Cu") (net 19))
   (segment (start 68.14805 60.80165) (end 66.2275 60.80165) (width 0.16) (layer "F.Cu") (net 19))
   (segment (start 69.0385 123.3021) (end 67.581 121.8446) (width 0.16) (layer "F.Cu") (net 19))
-  (segment (start 70.111 91.9646) (end 71.3212 91.9646) (width 0.16) (layer "F.Cu") (net 19))
   (segment (start 70.181 121.8446) (end 69.511 121.1746) (width 0.16) (layer "F.Cu") (net 19))
-  (segment (start 71.3212 91.9646) (end 71.3466 91.99) (width 0.16) (layer "F.Cu") (net 19))
   (segment (start 71.381 121.8446) (end 70.181 121.8446) (width 0.16) (layer "F.Cu") (net 19))
   (segment (start 71.381 121.8446) (end 67.581 121.8446) (width 0.16) (layer "F.Cu") (net 19))
   (segment (start 72.456 123.4446) (end 72.456 122.9196) (width 0.16) (layer "F.Cu") (net 19))
-  (via (at 70.111 91.9646) (size 0.8) (drill 0.4) (layers "F.Cu" "B.Cu") (net 19))
+  (via (at 72.0261 95.07) (size 0.8) (drill 0.4) (layers "F.Cu" "B.Cu") (net 19))
   (via (at 68.461 61.1146) (size 0.8) (drill 0.4) (layers "F.Cu" "B.Cu") (net 19))
   (via (at 69.511 121.1746) (size 0.8) (drill 0.4) (layers "F.Cu" "B.Cu") (net 19))
-  (segment (start 68.880989 100.414611) (end 71.061 98.2346) (width 0.16) (layer "B.Cu") (net 19))
-  (segment (start 68.461 90.3146) (end 68.461 61.1146) (width 0.16) (layer "B.Cu") (net 19))
-  (segment (start 71.061 92.9146) (end 70.111 91.9646) (width 0.16) (layer "B.Cu") (net 19))
-  (segment (start 68.880989 113.626064) (end 68.880989 100.414611) (width 0.16) (layer "B.Cu") (net 19))
-  (segment (start 71.061 98.2346) (end 71.061 92.9146) (width 0.16) (layer "B.Cu") (net 19))
-  (segment (start 69.279036 114.024111) (end 68.880989 113.626064) (width 0.16) (layer "B.Cu") (net 19))
-  (segment (start 69.660511 114.024111) (end 69.279036 114.024111) (width 0.16) (layer "B.Cu") (net 19))
-  (segment (start 70.111 91.9646) (end 68.461 90.3146) (width 0.16) (layer "B.Cu") (net 19))
-  (segment (start 69.511 121.1746) (end 69.660511 121.025089) (width 0.16) (layer "B.Cu") (net 19))
-  (segment (start 69.660511 121.025089) (end 69.660511 114.024111) (width 0.16) (layer "B.Cu") (net 19))
+  (segment (start 68.880989 113.626064) (end 69.279036 114.024111) (width 0.16) (layer "B.Cu") (net 19))
+  (segment (start 69.279036 114.024111) (end 69.660511 114.024111) (width 0.16) (layer "B.Cu") (net 19))
+  (segment (start 68.880989 100.414611) (end 68.880989 113.626064) (width 0.16) (layer "B.Cu") (net 19))
+  (segment (start 72.0261 95.07) (end 71.061 96.0351) (width 0.16) (layer "B.Cu") (net 19))
+  (segment (start 71.33 93.902625) (end 68.461 91.033625) (width 0.16) (layer "B.Cu") (net 19))
+  (segment (start 71.061 98.2346) (end 68.880989 100.414611) (width 0.16) (layer "B.Cu") (net 19))
+  (segment (start 68.461 91.033625) (end 68.461 61.1146) (width 0.16) (layer "B.Cu") (net 19))
+  (segment (start 72.0261 95.07) (end 71.33 94.3739) (width 0.16) (layer "B.Cu") (net 19))
+  (segment (start 69.660511 114.024111) (end 69.660511 121.025089) (width 0.16) (layer "B.Cu") (net 19))
+  (segment (start 69.660511 121.025089) (end 69.511 121.1746) (width 0.16) (layer "B.Cu") (net 19))
+  (segment (start 71.061 96.0351) (end 71.061 98.2346) (width 0.16) (layer "B.Cu") (net 19))
+  (segment (start 71.33 94.3739) (end 71.33 93.902625) (width 0.16) (layer "B.Cu") (net 19))
   (segment (start 85.021 64.3746) (end 84.78395 64.61165) (width 0.16) (layer "F.Cu") (net 20))
   (segment (start 93.8985 52.8746) (end 94.521 52.8746) (width 0.16) (layer "F.Cu") (net 20))
@@
   (segment (start 69.661 100.9346) (end 69.661 109.9746) (width 0.16) (layer "B.Cu") (net 31))
   (segment (start 72.377011 117.132589) (end 72.390011 117.145589) (width 0.16) (layer "B.Cu") (net 31))
-  (segment (start 72.181 96.8246) (end 72.071 96.7146) (width 0.16) (layer "F.Cu") (net 32))
   (segment (start 77.351 96.8246) (end 72.181 96.8246) (width 0.16) (layer "F.Cu") (net 32))
   (segment (start 76.511 110.2546) (end 77.451 110.2546) (width 0.16) (layer "F.Cu") (net 32))
   (segment (start 77.361 96.8346) (end 77.351 96.8246) (width 0.16) (layer "F.Cu") (net 32))
   (segment (start 75.8114 111.962787) (end 75.8114 110.9542) (width 0.16) (layer "F.Cu") (net 32))
-  (segment (start 72.9335 90.1843) (end 72.2966 90.8212) (width 0.16) (layer "F.Cu") (net 32))
-  (segment (start 72.071 96.7146) (end 72.071 94.0906) (width 0.16) (layer "F.Cu") (net 32))
-  (segment (start 72.071 94.0906) (end 72.2966 93.865) (width 0.16) (layer "F.Cu") (net 32))
-  (segment (start 72.2966 90.8212) (end 72.2966 93.865) (width 0.16) (layer "F.Cu") (net 32))
+  (segment (start 71.3466 95.9902) (end 72.181 96.8246) (width 0.16) (layer "F.Cu") (net 32))
+  (segment (start 72.9335 90.1843) (end 72.9335 90.4031) (width 0.16) (layer "F.Cu") (net 32))
+  (segment (start 72.9335 90.4031) (end 71.3466 91.99) (width 0.16) (layer "F.Cu") (net 32))
+  (segment (start 71.3212 91.9646) (end 71.3466 91.99) (width 0.16) (layer "F.Cu") (net 32))
   (segment (start 75.8114 110.9542) (end 76.271 110.4946) (width 0.16) (layer "F.Cu") (net 32))
+  (segment (start 71.3466 91.99) (end 71.3466 95.9902) (width 0.16) (layer "F.Cu") (net 32))
   (segment (start 76.271 110.4946) (end 76.511 110.2546) (width 0.16) (layer "F.Cu") (net 32))
   (via (at 77.361 96.8346) (size 0.8) (drill 0.4) (layers "F.Cu" "B.Cu") (net 32))
@@
     (connect_pads (clearance 0.5))
     (min_thickness 0.254) (filled_areas_thickness no)
-    (fill yes (thermal_gap 0.508) (thermal_bridge_width 0.508))
+    (fill yes (thermal_gap 0.508) (thermal_bridge_width 0.508) (island_removal_mode 1) (island_area_min 0))
     (polygon
       (pts
