File: GlowHubPCB/GlowHubPCB.kicad_sch (KiCad schematic)
At the start: 31 parts, among them Q2 MMBT2222A, Q3 MMBT2222A, SW1 TS-1185EC-C-D-B, SW2 TS-1185EC-C-D-B, U2 ESP32-WROOM-32E (4MB), U5 CP2102-GMR, U6 BL1117-33CX

Commit message: added GlowHub PCB prototype
Parts:
- removed C22: 220uF 10V, Capacitor_SMD:CP_Elec_6.3x5.4, symbol Device:C_Polarized
- added C1: 10uF, Capacitor_SMD:C_0603_1608Metric_Pad1.08x0.95mm_HandSolder, symbol Device:10uF 0603
- added D9: Schottky, Diode_SMD:D_SOD-123, symbol Device:D_Schottky
- added F1: BSMD1812-300-16V, Fuse:Fuse_1812_4532Metric_Pad1.30x3.40mm_HandSolder, symbol Device:Fuse
- added J1: Conn_01x08, Connector_PinSocket_2.54mm:PinSocket_1x08_P2.54mm_Vertical, symbol Connector_Generic:Conn_01x08
- added Q1, Q10, Q11, Q4, Q5, Q6, Q7, Q8, Q9: AP40P05, Package_TO_SOT_SMD:SOT-23, symbol Transistor_FET:SK338P
- added RJ9: R-RJ11R06P-A800, R-RJ11R06P-A800:R-RJ11R06P-A800, symbol R-RJ11R06P-A800:PCB-6P6C-90
- RJ1, RJ2, RJ3, RJ4, RJ5, RJ6, RJ7, RJ8: value PCB-6P6C-90 -> R-RJ11R06P-A800
Connections:
- net +3V3: now also J1.6 (Pin_6), Q5.3 (D); no longer C17.2, U6.2 (Vout), U6.4 (Vout)
- net +5V: now also C1.1, D9.2 (A), F1.2, J1.8 (Pin_8); no longer RJ1.5, RJ2.5, RJ3.5, RJ4.5, RJ5.5, RJ6.5, RJ7.5, RJ8.5, USB1.A4B9 (VBUS), USB1.B4A9 (VBUS)
- net GND: now also C1.2, J1.7 (Pin_7), RJ9.4
- net IO12/MISO: now also J1.1 (Pin_1)
- net IO13/MOSI: now also J1.2 (Pin_2)
- net IO16/LED1: now also Q6.2 (S); no longer RJ1.4
- net IO17/LED2: now also Q9.2 (S); no longer RJ5.4
- net IO18/LED3: now also Q1.2 (S); no longer RJ2.4
- net IO19/LED4: now also Q7.2 (S); no longer RJ6.4
- net IO21/LED5: now also Q10.2 (S); no longer RJ3.4
- net IO22/LED6: now also Q4.2 (S); no longer RJ7.4
- net IO23/LED7: now also Q8.2 (S); no longer RJ4.4
- net IO25/A1/DAC1: now also J1.4 (Pin_4)
- net IO26/A0/DAC2: now also J1.5 (Pin_5)
- net IO27/LED8: now also Q11.2 (S); no longer RJ8.4
- net IO5: now also J1.3 (Pin_3)
- net IO33/BUTTON renamed IO33/TESTBUTTON
- new net: F1.1, USB1.A4B9 (VBUS), USB1.B4A9 (VBUS)
- new net: C17.2, Q5.2 (S), U6.2 (Vout), U6.4 (Vout)
- new net EXTERNAL 5V: D9.1 (K), RJ1.5, RJ2.5, RJ3.5, RJ4.5, RJ5.5, RJ6.5, RJ7.5, RJ8.5
- new net LED1 DATA OUT: Q1.3 (D), Q10.3 (D), Q11.3 (D), Q4.3 (D), Q6.3 (D), Q7.3 (D), Q8.3 (D), Q9.3 (D), RJ1.4, RJ2.4, RJ3.4, RJ4.4, RJ5.4, RJ6.4, RJ7.4, RJ8.4, RJ9.3
- new net RECEIVER 5V: Q1.1 (G), Q10.1 (G), Q11.1 (G), Q4.1 (G), Q5.1 (G), Q6.1 (G), Q7.1 (G), Q8.1 (G), Q9.1 (G), RJ9.2
Other:
- note added: "Pins"
- note added: "Receiver mode"
- note added: "Test animations button"
- note removed: "Switch animations button"
- moved on the sheet: C16, C17, RJ1, RJ2, RJ3, RJ4, RJ5, RJ6, RJ7, RJ8, U6

Commit message: updated pcb design (in progress)
Parts:
- removed C18: 1uF, Capacitor_SMD:C_0603_1608Metric_Pad1.08x0.95mm_HandSolder, symbol Device:1uF 0603
- removed C19: 0.1uF, Capacitor_SMD:C_0603_1608Metric_Pad1.08x0.95mm_HandSolder, symbol Device:0.1uF 0603
- removed C5: 10uF, Capacitor_SMD:C_0603_1608Metric_Pad1.08x0.95mm_HandSolder, symbol Device:10uF 0603
- removed MK1: ICS-43432, ICS-43432:MIC_ICS-43432, symbol ICS-43432:ICS-43432
- removed Q2, Q3: MMBT2222A, Package_TO_SOT_SMD:SOT-23, symbol MMBT2222A:MMBT2222A
- removed Q5: AP40P05, Package_TO_SOT_SMD:SOT-23, symbol Transistor_FET:SK338P
- removed R16: 100K, Resistor_SMD:R_0603_1608Metric_Pad0.98x0.95mm_HandSolder, symbol Device:100K 0603
- removed R17, R18, R20: 10K, Resistor_SMD:R_0603_1608Metric_Pad0.98x0.95mm_HandSolder, symbol Device:10K 0603
- removed SW1, SW2: TS-1185EC-C-D-B, TS-1185EC-C-D-B:TS-1185EC-C-D-B, symbol TS-1185EC-C-D-B:TS-1185EC-C-D-B
- added C?: 0.1uF, Capacitor_SMD:C_0603_1608Metric_Pad1.08x0.95mm_HandSolder, symbol Device:0.1uF 0603
- added C?: 10uF, Capacitor_SMD:C_0603_1608Metric_Pad1.08x0.95mm_HandSolder, symbol Device:10uF 0603
- added C? (x2): 1nF, Capacitor_SMD:C_0603_1608Metric_Pad1.08x0.95mm_HandSolder, symbol Device:10uF 0603
- added D? (x8): Schottky, Diode_SMD:D_SOD-123, symbol Device:D_Schottky
- added R? (x2): 220, Resistor_SMD:R_0603_1608Metric_Pad0.98x0.95mm_HandSolder, symbol Device:10K 0603
- added R? (x2): 10K, Resistor_SMD:R_0603_1608Metric_Pad0.98x0.95mm_HandSolder, symbol Device:10K 0603
- added R?: 470, Resistor_SMD:R_0603_1608Metric_Pad0.98x0.95mm_HandSolder, symbol Device:100K 0603
- added SW? (x3): TS-1185EC-C-D-B, TS-1185EC-C-D-B:TS-1185EC-C-D-B, symbol TS-1185EC-C-D-B:TS-1185EC-C-D-B
- added U?: GMA4030H11-F26, GMA4030H11-F26:GMA4030H11-F26, symbol GMA4030H11-F26:GMA4030H11-F26
- added U?: UMH3N, footprint:SC-70-6_L2.2-W1.3-P0.65-LS2.1-BR, symbol LCSC:UMH3N
Connections:
- net +3V3: now also C17.2, U6.2 (Vout), U6.4 (Vout), C?.2, C?.2, R?.2, R?.2, U?.1 (VDD)
- net DTR: now also U?.2 (B), U?.4 (E)
- net GND: now also C?.1, C?.1, C?.2, C?.2, SW?.1, SW?.1, SW?.1, U?.5 (GND), U?.6 (GND), U?.7 (GND), U?.8 (GND)
- net IO0: now also C?.1, R?.1, R?.2, U?.3 (C)
- net IO14/SCK: now also U?.3 (CLOCK)
- net IO15/WS: now also U?.2 (SELECT)
- net IO32/SD: now also U?.4 (DATA)
- net IO33/TESTBUTTON: now also SW?.2
- net LED1 DATA OUT: now also D?.1 (K); no longer Q1.3 (D), Q10.3 (D), Q11.3 (D), Q4.3 (D), Q7.3 (D), Q8.3 (D), Q9.3 (D), RJ2.4, RJ3.4, RJ4.4, RJ5.4, RJ6.4, RJ7.4, RJ8.4, RJ9.3
- net RESET: now also C?.1, R?.1, R?.2, U?.6 (C)
- net RTS: now also U?.1 (E), U?.5 (B)
- net RXD0: now also R?.1; no longer U5.26 (TXD)
- new net: R?.1, SW?.2 (x2)
- new net: R?.2, U5.26 (TXD)
- new net LED2 DATA OUT: D?.1 (K), Q9.3 (D), RJ2.4
- new net LED3 DATA OUT: D?.1 (K), Q1.3 (D), RJ3.4
- new net LED4 DATA OUT: D?.1 (K), Q7.3 (D), RJ4.4
- new net LED5 DATA OUT: D?.1 (K), Q10.3 (D), RJ5.4
- new net LED6 DATA OUT: D?.1 (K), Q4.3 (D), RJ6.4
- new net LED7 DATA OUT: D?.1 (K), Q8.3 (D), RJ7.4
- new net LED8 DATA OUT: D?.1 (K), Q11.3 (D), RJ8.4
- new net RECEIVER LED DATA: D?.2 (A), D?.2 (A), D?.2 (A), D?.2 (A), D?.2 (A), D?.2 (A), D?.2 (A), D?.2 (A), RJ9.3
Other:
- note added: "Auto program DTR RTS --> EN IO0 1 1 1 1 0 0 1 1 1 0 0 1 0 1 1 0"
- note removed: "3.3V step down"
- moved on the sheet: C16, C17, Q1, Q10, Q11, Q4, Q6, Q7, Q8, Q9, R1, R2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
